File: edge triggered monostable.kicad_pcb (KiCad board)
At the start: 2 copper layers, 77 x 23 mm, 14 parts, among them J1 Screw_Terminal_01x02, J2 Screw_Terminal_01x06, J3 Screw_Terminal_01x02, K1 G5V-2, U1 NE555D

Commit message: Added LED, BOM, and position files...
Parts:
- added D3: LED, LED_SMD:LED_0805_2012Metric, F.Cu at (122.9, 101.0)
- added R5: 1.5K, Resistor_SMD:R_0805_2012Metric, F.Cu at (122.9, 105.5)
- added REF**: MountingHole_2.5mm, MountingHole:MountingHole_2.5mm, F.Cu at (161.0, 111.0)
- added REF**: MountingHole_2.5mm, MountingHole:MountingHole_2.5mm, F.Cu at (86.0, 111.0)
- added REF**: MountingHole_2.5mm, MountingHole:MountingHole_2.5mm, F.Cu at (86.0, 90.0)
- added REF**: MountingHole_2.5mm, MountingHole:MountingHole_2.5mm, F.Cu at (161.0, 90.0)
- moved D2 1.68 mm to (121.5, 95.8)
Routing:
- net Net-(D2-A): track 24.7 -> 28.3 mm
- net Net-(D3-A): track 0.00 -> 2.66 mm
Other:
- board size 77 x 23 mm -> 82 x 28 mm
- board text added: "IN"
- board text removed: "In"

Commit message: First board release. Order has been placed.
Parts:
- removed J2: Screw_Terminal_01x06, TerminalBlock_Phoenix:TerminalBlock_Phoenix_MPT-0,5-6-2.54_1x06_P2.54mm_Horizontal
- added J4: Screw_Terminal_01x02, TerminalBlock_TE-Connectivity:TerminalBlock_TE_282834-2_1x02_P2.54mm_Horizontal, F.Cu at (153.5, 108.5)
- added J5: Screw_Terminal_01x02, TerminalBlock_TE-Connectivity:TerminalBlock_TE_282834-2_1x02_P2.54mm_Horizontal, F.Cu at (153.5, 101.8)
- added J6: Screw_Terminal_01x02, TerminalBlock_TE-Connectivity:TerminalBlock_TE_282834-2_1x02_P2.54mm_Horizontal, F.Cu at (153.5, 95.0)
- J1, J3: footprint TerminalBlock_Phoenix:TerminalBlock_Phoenix_MPT-0,5-2-2.54_1x02_P2.54mm_Horizontal -> TerminalBlock_TE-Connectivity:TerminalBlock_TE_282834-2_1x02_P2.54mm_Horizontal
- moved REF** 3.00 mm to (164.0, 111.0)
- moved REF** 3.00 mm to (164.0, 90.0)
- moved REF** 2.00 mm to (84.0, 111.0)
- moved REF** 2.00 mm to (84.0, 90.0)
Routing:
- net Net-(J4-Pin_1): track 16.1 -> 13.9 mm
- net Net-(J4-Pin_2): track 10.2 -> 8.40 mm
- net Net-(J5-Pin_1): track 21.4 -> 20.3 mm
- net Net-(J5-Pin_2): track 15.7 -> 14.7 mm
Other:
- board size 82 x 28 mm -> 86.8 x 28 mm
