File: edge triggered monostable.kicad_sch (KiCad schematic)
At the start: 14 parts, among them J1 Screw_Terminal_01x02, J2 Screw_Terminal_01x06, J3 Screw_Terminal_01x02, K1 G5V-2, U1 NE555D

Commit message: Added LED, BOM, and position files...
Parts:
- added D3: LED, LED_SMD:LED_0805_2012Metric, symbol Device:LED
- added R5: 1.5K, Resistor_SMD:R_0805_2012Metric, symbol Device:R
- C1: LCSC (none) -> C440198
- C2, C3: LCSC (none) -> C49678
- D1, D2: LCSC (none) -> C81598
- J1, J3: LCSC (none) -> C557685
- J2: LCSC (none) -> C915915
- K1: LCSC (none) -> C28089
- R1: LCSC (none) -> C17514
- R2, R3, R4: LCSC (none) -> C17414
- U1: LCSC (none) -> C7593
Connections:
- net +12V: now also R5.1
- net at D2.2 (A), K1.16, U1.3 (Q): now also D3.1 (K)
- new net: D3.2 (A), R5.2
Other:
- moved on the sheet: C1, C2, C3, D1, D2, J1, J2, J3, K1, R1, R2, R3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

Commit message: First board release. Order has been placed.
Parts:
- removed J2: Screw_Terminal_01x06, TerminalBlock_Phoenix:TerminalBlock_Phoenix_MPT-0,5-6-2.54_1x06_P2.54mm_Horizontal, symbol Connector:Screw_Terminal_01x06
- added J4, J5, J6: Screw_Terminal_01x02, TerminalBlock_TE-Connectivity:TerminalBlock_TE_282834-2_1x02_P2.54mm_Horizontal, symbol Connector:Screw_Terminal_01x02
- J1, J3: footprint TerminalBlock_Phoenix:TerminalBlock_Phoenix_MPT-0,5-2-2.54_1x02_P2.54mm_Horizontal -> TerminalBlock_TE-Connectivity:TerminalBlock_TE_282834-2_1x02_P2.54mm_Horizontal; LCSC C557685 -> C2922597
Connections:
- net at K1.6: now also J4.1 (Pin_1)
- net at K1.8: now also J4.2 (Pin_2)
- net at K1.4: now also J5.1 (Pin_1)
- net at K1.11: now also J5.2 (Pin_2)
- net at K1.9: now also J6.1 (Pin_1)
- net at K1.13: now also J6.2 (Pin_2)
Changed lines of the file:
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@@
     )
   )
-  (symbol (lib_id "Connector:Screw_Terminal_01x06") (at 234.95 83.82 0) (unit 1)
-    (in_bom yes) (on_board yes) (dnp no)
-    (property "Reference" "J2" (at 234.95 95.25 0)
-      (effects (font (size 1.27 1.27)) (justify left))
-    )
-    (property "Value" "Screw_Terminal_01x06" (at 234.95 97.79 0)
-      (effects (font (size 1.27 1.27)) (justify left))
-    )
-    (property "Footprint" "TerminalBlock_Phoenix:TerminalBlock_Phoenix_MPT-0,5-6-2.54_1x06_P2.54mm_Horizontal" (at 234.95 83.82 0)
+  (symbol (lib_id "Connector:Screw_Terminal_01x02") (at 234.95 83.82 0) (unit 1)
+    (in_bom yes) (on_board yes) (dnp no)
+    (property "Reference" "J5" (at 238.76 83.82 0)
+      (effects (font (size 1.27 1.27)))
+    )
+    (property "Value" "Screw_Terminal_01x02" (at 243.84 90.17 0)
+      (effects (font (size 1.27 1.27)) hide)
+    )
+    (property "Footprint" "TerminalBlock_TE-Connectivity:TerminalBlock_TE_282834-2_1x02_P2.54mm_Horizontal" (at 234.95 83.82 0)
       (effects (font (size 1.27 1.27)) hide)
     )
@@
       (effects (font (size 1.27 1.27)) hide)
     )
-    (property "LCSC" "C915915" (at 234.95 83.82 0)
-      (effects (font (size 1.27 1.27)) hide)
-    )
-    (pin "1")
-    (pin "2")
-    (pin "3")
-    (pin "4")
-    (pin "5")
-    (pin "6")
-    (instances
-      (project "edge triggered monostable"
-        (path "/bc524914-33a0-4e61-87c8-1952b08088d4"
-          (reference "J2") (unit 1)
+    (property "LCSC" "    C2922597" (at 234.95 83.82 0)
+      (effects (font (size 1.27 1.27)) hide)
+    )
+    (pin "1")
+    (pin "2")
+    (instances
+      (project "edge triggered monostable"
+        (path "/bc524914-33a0-4e61-87c8-1952b08088d4"
+          (reference "J5") (unit 1)
         )
       )
@@
         (path "/bc524914-33a0-4e61-87c8-1952b08088d4"
           (reference "U1") (unit 1)
+        )
+      )
+    )
+  )
+  (symbol (lib_id "Connector:Screw_Terminal_01x02") (at 234.95 88.9 0) (unit 1)
+    (in_bom yes) (on_board yes) (dnp no)
+    (property "Reference" "J6" (at 238.76 88.9 0)
+      (effects (font (size 1.27 1.27)))
+    )
+    (property "Value" "Screw_Terminal_01x02" (at 243.84 95.25 0)
+      (effects (font (size 1.27 1.27)) hide)
+    )
+    (property "Footprint" "TerminalBlock_TE-Connectivity:TerminalBlock_TE_282834-2_1x02_P2.54mm_Horizontal" (at 234.95 88.9 0)
+      (effects (font (size 1.27 1.27)) hide)
+    )
+    (property "Datasheet" "~" (at 234.95 88.9 0)
+      (effects (font (size 1.27 1.27)) hide)
+    )
+    (property "LCSC" "    C2922597" (at 234.95 88.9 0)
+      (effects (font (size 1.27 1.27)) hide)
+    )
+    (pin "1")
+    (pin "2")
+    (instances
+      (project "edge triggered monostable"
+        (path "/bc524914-33a0-4e61-87c8-1952b08088d4"
+          (reference "J6") (unit 1)
         )
       )
@@
   (symbol (lib_id "Connector:Screw_Terminal_01x02") (at 62.23 115.57 0) (mirror y) (unit 1)
     (in_bom yes) (on_board yes) (dnp no)
-    (property "Reference" "J1" (at 53.34 124.46 0)
+    (property "Reference" "J1" (at 58.42 115.57 0)
       (effects (font (size 1.27 1.27)))
     )
     (property "Value" "Screw_Terminal_01x02" (at 53.34 121.92 0)
-      (effects (font (size 1.27 1.27)))
-    )
-    (property "Footprint" "TerminalBlock_Phoenix:TerminalBlock_Phoenix_MPT-0,5-2-2.54_1x02_P2.54mm_Horizontal" (at 62.23 115.57 0)
+      (effects (font (size 1.27 1.27)) hide)
+    )
+    (property "Footprint" "TerminalBlock_TE-Connectivity:TerminalBlock_TE_282834-2_1x02_P2.54mm_Horizontal" (at 62.23 115.57 0)
       (effects (font (size 1.27 1.27)) hide)
     )
@@
       (effects (font (size 1.27 1.27)) hide)
     )
-    (property "LCSC" "C557685" (at 62.23 115.57 0)
+    (property "LCSC" "    C2922597" (at 62.23 115.57 0)
       (effects (font (size 1.27 1.27)) hide)
     )
@@
   (symbol (lib_id "Connector:Screw_Terminal_01x02") (at 62.23 82.55 0) (mirror y) (unit 1)
     (in_bom yes) (on_board yes) (dnp no)
-    (property "Reference" "J3" (at 53.34 91.44 0)
+    (property "Reference" "J3" (at 58.42 82.55 0)
       (effects (font (size 1.27 1.27)))
     )
     (property "Value" "Screw_Terminal_01x02" (at 53.34 88.9 0)
-      (effects (font (size 1.27 1.27)))
-    )
-    (property "Footprint" "TerminalBlock_Phoenix:TerminalBlock_Phoenix_MPT-0,5-2-2.54_1x02_P2.54mm_Horizontal" (at 62.23 82.55 0)
+      (effects (font (size 1.27 1.27)) hide)
+    )
+    (property "Footprint" "TerminalBlock_TE-Connectivity:TerminalBlock_TE_282834-2_1x02_P2.54mm_Horizontal" (at 62.23 82.55 0)
       (effects (font (size 1.27 1.27)) hide)
     )
@@
       (effects (font (size 1.27 1.27)) hide)
     )
-    (property "LCSC" "C557685" (at 62.23 82.55 0)
+    (property "LCSC" "    C2922597" (at 62.23 82.55 0)
       (effects (font (size 1.27 1.27)) hide)
     )
@@
         )
       )
+    )
+  )
+  (symbol (lib_id "Connector:Screw_Terminal_01x02") (at 234.95 78.74 0) (unit 1)
+    (in_bom yes) (on_board yes) (dnp no)
+    (property "Reference" "J4" (at 238.76 78.74 0)
+      (effects (font (size 1.27 1.27)))
+    )
+    (property "Value" "Screw_Terminal_01x02" (at 243.84 85.09 0)
+      (effects (font (size 1.27 1.27)) hide)
+    )
+    (property "Footprint" "TerminalBlock_TE-Connectivity:TerminalBlock_TE_282834-2_1x02_P2.54mm_Horizontal" (at 234.95 78.74 0)
+      (effects (font (size 1.27 1.27)) hide)
+    )
+    (property "Datasheet" "~" (at 234.95 78.74 0)
+      (effects (font (size 1.27 1.27)) hide)
+    )
+    (property "LCSC" "    C2922597" (at 234.95 78.74 0)
+      (effects (font (size 1.27 1.27)) hide)
+    )
+    (pin "1")
+    (pin "2")
+    (instances
+      (project "edge triggered monostable"
+        (path "/bc524914-33a0-4e61-87c8-1952b08088d4"
+          (reference "J4") (unit 1)
+        )
+      )
